File: knob.kicad_pcb (KiCad board)
At the start: 2 copper layers, 35 x 19 mm, 8 parts, among them J1 SJ2-35464B-SMT-TR

Commit message: Update Library
Parts:
- FID1, FID101, FID102: value Fiducial -> Fiducial_Paste
- H1, H2: value MountingHole_2.5mm -> 2.5mm
- RV101: value 10k -> 50R
Connections:
- RV101 pad 4: (no net) -> unconnected-(RV101-SW1-Pad4)
- RV101 pad 5: (no net) -> unconnected-(RV101-Pad5)
